File: Schematic/System/Anenometer.sch (KiCad schematic (older format))
At the start: 0 parts

Commit message: Schematic project reset
Changed lines of the file:
@@
 $Descr A4 11693 8268
 encoding utf-8
-Sheet 4 9
+Sheet 9 14
 Title ""
 Date ""
@@
 $EndDescr
 $Sheet
-S 1600 1200 1450 1700
-U 5C8D1F09
+S 2350 2600 2050 1950
+U 5C8F8359
 F0 "Control Board" 50
 F1 "Control.sch" 50
 $EndSheet
 $Sheet
-S 4550 1200 1450 1750
-U 5C8D1FD1
-F0 "Switch Board" 50
-F1 "SWBoard.sch" 50
+S 6850 2250 700  650
+U 5C8F8445
+F0 "North Tx Rx" 50
+F1 "N_TxRx.sch" 50
 $EndSheet
 $Sheet
-S 7400 1200 1300 1750
-U 5C8D20C3
-F0 "Sensor Board" 50
-F1 "SenBoard.sch" 50
+S 5700 3200 700  650
+U 5C8F86DD
+F0 "West Tx Rx" 50
+F1 "W_TxRx.sch" 50
+$EndSheet
+$Sheet
+S 6850 4050 700  650
+U 5C8F8711
+F0 "South Tx Rx" 50
+F1 "S_TxRx.sch" 50
+$EndSheet
+$Sheet
+S 7950 3200 700  650
+U 5C8F8793
+F0 "East Tx Rx" 50
+F1 "E_TxRx.sch" 50
 $EndSheet
 $EndSCHEMATC
