File: Schematic/System/IntPSU.sch (KiCad schematic (older format))
At the start: 0 parts

Commit message: Schematic project reset
Connections:
- net labels removed: +12v
- wire segments 1 -> 0
Changed lines of the file:
@@
 $Descr A4 11693 8268
 encoding utf-8
-Sheet 2 9
+Sheet 1 14
 Title ""
 Date ""
@@
 Comment4 ""
 $EndDescr
-Text HLabel 1900 1800 0    50   Input ~ 0
-+12v
-Wire Wire Line
-	2100 1800 1900 1800
 $EndSCHEMATC
