File: Schematic/System/N_TxRx.sch (KiCad schematic (older format))
At the start: 17 parts

Commit message: Start board layout
Parts:
- removed R?: R, symbol Device:R
- added R2, R9: R, Resistor_THT:R_Axial_DIN0207_L6.3mm_D2.5mm_P7.62mm_Horizontal, symbol Device:R
- D1, D2: renamed from D?; footprint (none) -> Diode_THT:D_DO-35_SOD27_P7.62mm_Horizontal
- R1, R10, R11, R12, R3, R4, R5, R6, R7, R8: renamed from R?; footprint (none) -> Resistor_THT:R_Axial_DIN0207_L6.3mm_D2.5mm_P7.62mm_Horizontal
- gave numbers to parts that had none: 4
Connections:
- net at U1.1 (+): now also R6.2, R9.2
- net GND: now reaches U1.2 (V-)
- net GND: now also Q1.2 (S), R10.2, R12.1, R4.1, R8.2, R9.1
- net at U1.3 (-): now also D1.1 (K), D2.2 (A)
- net at U1.4: now also R2.1
- net +5V: now reaches U1.5 (V+)
- net +5V: now also R6.1
- net at Q2.1 (G): now also R3.2, R5.1
- net +28V: now reaches Q2.2 (S)
- net +28V: now also R3.1
- net at Q2.3 (D): now also Q3.2 (S), R11.1, R12.2, R7.1
- net at Q3.1 (G): now also R7.2, R8.1
- net at Q3.3 (D): now also R10.1
- net at Q1.1 (G): now also R1.1, R4.2
- net at Q1.3 (D): now also R5.2
- net at R11.2: now also D1.2 (A), D2.1 (K)
- new net NorthRxOutput: R2.2
Other:
- moved on the sheet: D1, D2, Q2, Q3, R10, R11, R12, R3, R4, R5, R6, R7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
