File: Schematic/System/System.sch (KiCad schematic (older format))
At the start: 0 parts

Commit message: schematic changes
Changed lines of the file:
@@
 $EndSheet
 $Sheet
-S 3900 3800 900  1300
+S 3800 3800 900  1300
 U 5C8D1A7C
 F0 "Anenometer" 50

Commit message: Schematic project reset
Changed lines of the file:
@@
 $Descr A4 11693 8268
 encoding utf-8
-Sheet 1 9
+Sheet 1 14
 Title ""
 Date ""
@@
 $EndDescr
 $Sheet
-S 1950 1400 1400 1400
-U 5C8D0D73
-F0 "Power Supply" 50
-F1 "PSU.sch" 50
-F2 "+12v" I R 3350 1700 50
+S 1600 1200 1050 1050
+U 5C8F7B4E
+F0 "External Power Supply" 50
+F1 "ExtPSU.sch" 50
 $EndSheet
 $Sheet
-S 1950 3800 850  1250
-U 5C8D19DC
-F0 "Rain" 50
-F1 "Rain.sch" 50
+S 1650 3200 950  1050
+U 5C8F7C88
+F0 "Internal Power Supply" 50
+F1 "IntPSU.sch" 50
 $EndSheet
 $Sheet
-S 3800 3800 900  1300
-U 5C8D1A7C
-F0 "Anenometer" 50
+S 3450 1200 900  1050
+U 5C8F7D5D
+F0 "External ESP8266" 50
+F1 "ExtMCU.sch" 50
+$EndSheet
+$Sheet
+S 3500 3100 800  1100
+U 5C8F7DEC
+F0 "Internal ESP8266" 50
+F1 "IntMCU.sch" 50
+$EndSheet
+$Sheet
+S 5150 1150 1100 1100
+U 5C8F7E91
+F0 "External Temp/Hum Sensor" 50
+F1 "THSenExt.sch" 50
+$EndSheet
+$Sheet
+S 5200 3100 1100 1100
+U 5C8F7F8F
+F0 "Internal Temp/Hum Sensor" 50
+F1 "THSenInt.sch" 50
+$EndSheet
+$Sheet
+S 6950 1150 900  1100
+U 5C8F8005
+F0 "Rain Fall Sensor" 50
+F1 "RainSen.sch" 50
+$EndSheet
+$Sheet
+S 8500 1150 1000 1100
+U 5C8F80D4
+F0 "Anenometer Sensor" 50
 F1 "Anenometer.sch" 50
 $EndSheet
-$Sheet
-S 5750 3800 900  1300
-U 5C8D1B69
-F0 "Temperature and Humidity" 50
-F1 "TempHum.sch" 50
-$EndSheet
-$Sheet
-S 5700 1350 2200 1500
-U 5C8D1CB2
-F0 "Comunication" 50
-F1 "coms.sch" 50
-$EndSheet
 $EndSCHEMATC

Commit message: Start board layout
Changed lines of the file:
@@
 $EndSheet
 $Sheet
-S 1650 3200 950  1050
+S 1750 4850 950  1050
 U 5C8F7C88
 F0 "Internal Power Supply" 50
@@
 $EndSheet
 $Sheet
-S 3500 3100 800  1100
+S 3600 4750 800  1100
 U 5C8F7DEC
 F0 "Internal ESP8266" 50
@@
 $EndSheet
 $Sheet
-S 5200 3100 1100 1100
+S 5300 4750 1100 1100
 U 5C8F7F8F
 F0 "Internal Temp/Hum Sensor" 50
@@
 $EndSheet
 $Sheet
-S 6950 1150 900  1100
+S 7000 1200 900  1100
 U 5C8F8005
 F0 "Rain Fall Sensor" 50
@@
 $EndSheet
 $Sheet
-S 8500 1150 1000 1100
+S 8700 1200 1000 1100
 U 5C8F80D4
 F0 "Anenometer Sensor" 50
