File: Schematic/Weather/Ext_MCU.sch (KiCad schematic (older format))
At the start: 0 parts

Commit message: More Board Data
Parts:
- added J?: 4_Way_Wire, symbol MyComponents:4_Way_Wire
- added U?: ESP-01v090, symbol ESP8266:ESP-01v090
- added U?: AMS1117, symbol MyComponents:AMS1117
Connections:
- net labels added: J10_P1, J10_P3, J10_P4, J10_p2, J8_P1, J8_P2, J8_P3, J8_P4, J9_P1, J9_P2, J9_P3, J9_P4
- wire segments 0 -> 12
Changed lines of the file:
@@
 EESchema Schematic File Version 4
+LIBS:Weather-cache
 EELAYER 29 0
 EELAYER END
 $Descr A4 11693 8268
 encoding utf-8
-Sheet 1 7
+Sheet 7 10
 Title ""
 Date ""
@@
 Comment4 ""
 $EndDescr
+Text HLabel 2650 3100 0    50   Input ~ 0
+J8_P1
+Text HLabel 2650 3300 0    50   Input ~ 0
+J8_P2
+Text HLabel 2650 3500 0    50   Input ~ 0
+J8_P3
+Text HLabel 2650 3700 0    50   Input ~ 0
+J8_P4
+Text HLabel 7850 2650 0    50   Input ~ 0
+J9_P1
+Text HLabel 7850 2850 0    50   Input ~ 0
+J9_P2
+Text HLabel 7850 3050 0    50   Input ~ 0
+J9_P3
+Text HLabel 7850 3250 0    50   Input ~ 0
+J9_P4
+Text HLabel 7850 3650 0    50   Input ~ 0
+J10_P1
+Text HLabel 7850 3850 0    50   Input ~ 0
+J10_p2
+Text HLabel 7850 4050 0    50   Input ~ 0
+J10_P3
+Text HLabel 7850 4250 0    50   Input ~ 0
+J10_P4
+$Comp
+L ESP8266:ESP-01v090 U?
+U 1 1 5C950A1B
+P 5550 3650
+F 0 "U?" H 5550 4165 50  0000 C CNN
+F 1 "ESP-01v090" H 5550 4074 50  0000 C CNN
+F 2 "" H 5550 3650 50  0001 C CNN
+F 3 "http://l0l.org.uk/2014/12/esp8266-modules-hardware-guide-gotta-catch-em-all/" H 5550 3650 50  0001 C CNN
+	1    5550 3650
+	1    0    0    -1
+$EndComp
+$Comp
+L MyComponents:4_Way_Wire J?
+U 1 1 5C964519
+P 3100 3100
+F 0 "J?" H 3050 2350 50  0000 L CNN
+F 1 "4_Way_Wire" H 2850 2200 50  0000 L CNN
+F 2 "" H 3000 3150 50  0001 C CNN
+F 3 "" H 3000 3150 50  0001 C CNN
+	1    3100 3100
+	1    0    0    -1
+$EndComp
+$Comp
+L MyComponents:AMS1117 U?
+U 1 1 5C951D08
+P 3200 1950
+F 0 "U?" V 2700 2000 60  0000 R CNN
+F 1 "AMS1117" V 2600 2200 60  0000 R CNN
+F 2 "" H 3200 1950 60  0000 C CNN
+F 3 "" H 3200 1950 60  0000 C CNN
+	1    3200 1950
+	0    -1   -1   0
+$EndComp
+Wire Wire Line
+	6500 3500 6500 2850
+Wire Wire Line
+	6500 2850 3650 2850
+Wire Wire Line
+	3100 2850 3100 3100
+Wire Wire Line
+	3650 2200 3650 2850
+Connection ~ 3650 2850
+Wire Wire Line
+	3650 2850 3100 2850
+Wire Wire Line
+	3650 1700 4000 1700
+Wire Wire Line
+	4000 1700 4000 3600
+Wire Wire Line
+	4000 3600 3100 3600
+Wire Wire Line
+	3100 3600 3100 3700
+Wire Wire Line
+	3650 1950 4300 1950
+Wire Wire Line
+	4300 1950 4300 3800
+Wire Wire Line
+	4300 3800 4600 3800
 $EndSCHEMATC

Commit message: North TxRx diode change
Parts:
- U?: symbol ESP8266:ESP-01v090 -> Weather-rescue:ESP-01v090-ESP8266
Changed lines of the file:
@@
 J10_P4
 $Comp
-L ESP8266:ESP-01v090 U?
+L Weather-rescue:ESP-01v090-ESP8266 U?
 U 1 1 5C950A1B
 P 5550 3650
+AR Path="/5C950A1B" Ref="U?"  Part="1"
+AR Path="/5C93D4CF/5C950A1B" Ref="U?"  Part="1"
 F 0 "U?" H 5550 4165 50  0000 C CNN
 F 1 "ESP-01v090" H 5550 4074 50  0000 C CNN

Commit message: schematic changes
Parts:
- gave numbers to parts that had none: 3
Changed lines of the file:
@@
 P 5550 3650
 AR Path="/5C950A1B" Ref="U?"  Part="1"
-AR Path="/5C93D4CF/5C950A1B" Ref="U?"  Part="1"
-F 0 "U?" H 5550 4165 50  0000 C CNN
+AR Path="/5C93D4CF/5C950A1B" Ref="U4"  Part="1"
+F 0 "U4" H 5550 4165 50  0000 C CNN
 F 1 "ESP-01v090" H 5550 4074 50  0000 C CNN
 F 2 "" H 5550 3650 50  0001 C CNN
@@
 $EndComp
 $Comp
-L MyComponents:4_Way_Wire J?
+L MyComponents:4_Way_Wire J1
 U 1 1 5C964519
 P 3100 3100
-F 0 "J?" H 3050 2350 50  0000 L CNN
+F 0 "J1" H 3050 2350 50  0000 L CNN
 F 1 "4_Way_Wire" H 2850 2200 50  0000 L CNN
 F 2 "" H 3000 3150 50  0001 C CNN
@@
 $EndComp
 $Comp
-L MyComponents:AMS1117 U?
+L MyComponents:AMS1117 U3
 U 1 1 5C951D08
 P 3200 1950
-F 0 "U?" V 2700 2000 60  0000 R CNN
+F 0 "U3" V 2700 2000 60  0000 R CNN
 F 1 "AMS1117" V 2600 2200 60  0000 R CNN
 F 2 "" H 3200 1950 60  0000 C CNN

Commit message: Start PCB
Parts:
- J1: footprint (none) -> Connector_PinHeader_2.54mm:PinHeader_1x04_P2.54mm_Vertical
- U3: footprint (none) -> Package_TO_SOT_SMD:SOT-223-3_TabPin2
- U4: footprint (none) -> footprint:ESP-01
Changed lines of the file:
@@
 F 0 "U4" H 5550 4165 50  0000 C CNN
 F 1 "ESP-01v090" H 5550 4074 50  0000 C CNN
-F 2 "" H 5550 3650 50  0001 C CNN
+F 2 "footprint:ESP-01" H 5550 3650 50  0001 C CNN
 F 3 "http://l0l.org.uk/2014/12/esp8266-modules-hardware-guide-gotta-catch-em-all/" H 5550 3650 50  0001 C CNN
 	1    5550 3650
@@
 F 0 "J1" H 3050 2350 50  0000 L CNN
 F 1 "4_Way_Wire" H 2850 2200 50  0000 L CNN
-F 2 "" H 3000 3150 50  0001 C CNN
+F 2 "Connector_PinHeader_2.54mm:PinHeader_1x04_P2.54mm_Vertical" H 3000 3150 50  0001 C CNN
 F 3 "" H 3000 3150 50  0001 C CNN
 	1    3100 3100
@@
 F 0 "U3" V 2700 2000 60  0000 R CNN
 F 1 "AMS1117" V 2600 2200 60  0000 R CNN
-F 2 "" H 3200 1950 60  0000 C CNN
+F 2 "Package_TO_SOT_SMD:SOT-223-3_TabPin2" H 3200 1950 60  0001 C CNN
 F 3 "" H 3200 1950 60  0000 C CNN
 	1    3200 1950
