File: Schematic/Weather/N_Sen.sch (KiCad schematic (older format))
At the start: 20 parts, among them Q1 BSS138, Q2 AO3401, Q3 AO3401, U1 LM321

Commit message: North TxRx diode change
Parts:
- added C?: C, symbol Device:C
- D1, D2: value D -> in916
- Q2, Q3: symbol Transistor_FET:AO3401 -> Weather-rescue:AO3401-Transistor_FET
- R1: value R -> 2.2K
- R10: value R -> 680
- R11: value R -> 3.3k
- R12: value R -> 47K
- R2, R6, R9: value R -> 4.7K
- R3: value R -> 2.2k
- R4: value R -> 5.1K
- R5: value R -> 10K
- R7, R8: value R -> 20K
Connections:
- net labels added: 0v, 24v, 5v
- wire segments 70 -> 73
Other:
- moved on the sheet: D1, D2, R11, R2, R6, R9, U1
Changed lines of the file:
@@
 J17_P8
 $Comp
-L Transistor_FET:AO3401 Q2
+L Weather-rescue:AO3401-Transistor_FET Q2
 U 1 1 5C8F913C
 P 6300 3600
@@
 L Amplifier_Operational:LM321 U1
 U 1 1 5C8F90C7
-P 6300 2150
-F 0 "U1" H 6300 2631 50  0000 C CNN
-F 1 "LM321" H 6300 2540 50  0000 C CNN
-F 2 "Package_TO_SOT_SMD:SOT-23-5" H 6300 2150 50  0001 C CNN
-F 3 "http://www.ti.com/lit/ds/symlink/lm321.pdf" H 6300 2150 50  0001 C CNN
-	1    6300 2150
+P 6050 2150
+F 0 "U1" H 6050 2631 50  0000 C CNN
+F 1 "LM321" H 6050 2540 50  0000 C CNN
+F 2 "Package_TO_SOT_SMD:SOT-23-5" H 6050 2150 50  0001 C CNN
+F 3 "http://www.ti.com/lit/ds/symlink/lm321.pdf" H 6050 2150 50  0001 C CNN
+	1    6050 2150
 	-1   0    0    -1
 $EndComp
@@
 P 5450 4800
 F 0 "R1" V 5243 4800 50  0000 C CNN
-F 1 "R" V 5334 4800 50  0000 C CNN
+F 1 "2.2K" V 5334 4800 50  0000 C CNN
 F 2 "Resistor_THT:R_Axial_DIN0207_L6.3mm_D2.5mm_P7.62mm_Horizontal" V 5380 4800 50  0001 C CNN
 F 3 "~" H 5450 4800 50  0001 C CNN
@@
 P 5850 5250
 F 0 "R4" H 5780 5204 50  0000 R CNN
-F 1 "R" H 5780 5295 50  0000 R CNN
+F 1 "5.1K" H 5780 5295 50  0000 R CNN
 F 2 "Resistor_THT:R_Axial_DIN0207_L6.3mm_D2.5mm_P7.62mm_Horizontal" V 5780 5250 50  0001 C CNN
 F 3 "~" H 5850 5250 50  0001 C CNN
@@
 P 7350 4900
 F 0 "R10" H 7420 4946 50  0000 L CNN
-F 1 "R" H 7420 4855 50  0000 L CNN
+F 1 "680" H 7420 4855 50  0000 L CNN
 F 2 "Resistor_THT:R_Axial_DIN0207_L6.3mm_D2.5mm_P7.62mm_Horizontal" V 7280 4900 50  0001 C CNN
 F 3 "~" H 7350 4900 50  0001 C CNN
@@
 P 7050 3900
 F 0 "R7" H 7120 3946 50  0000 L CNN
-F 1 "R" H 7120 3855 50  0000 L CNN
+F 1 "20K" H 7120 3855 50  0000 L CNN
 F 2 "Resistor_THT:R_Axial_DIN0207_L6.3mm_D2.5mm_P7.62mm_Horizontal" V 6980 3900 50  0001 C CNN
 F 3 "~" H 7050 3900 50  0001 C CNN
@@
 P 7700 3800
 F 0 "R12" H 7770 3846 50  0000 L CNN
-F 1 "R" H 7770 3755 50  0000 L CNN
+F 1 "47K" H 7770 3755 50  0000 L CNN
 F 2 "Resistor_THT:R_Axial_DIN0207_L6.3mm_D2.5mm_P7.62mm_Horizontal" V 7630 3800 50  0001 C CNN
 F 3 "~" H 7700 3800 50  0001 C CNN
@@
 P 6300 4150
 F 0 "R5" H 6370 4196 50  0000 L CNN
-F 1 "R" H 6370 4105 50  0000 L CNN
+F 1 "10K" H 6370 4105 50  0000 L CNN
 F 2 "Resistor_THT:R_Axial_DIN0207_L6.3mm_D2.5mm_P7.62mm_Horizontal" V 6230 4150 50  0001 C CNN
 F 3 "~" H 6300 4150 50  0001 C CNN
@@
 P 5750 3750
 F 0 "R3" H 5820 3796 50  0000 L CNN
-F 1 "R" H 5820 3705 50  0000 L CNN
+F 1 "2.2k" H 5820 3705 50  0000 L CNN
 F 2 "Resistor_THT:R_Axial_DIN0207_L6.3mm_D2.5mm_P7.62mm_Horizontal" V 5680 3750 50  0001 C CNN
 F 3 "~" H 5750 3750 50  0001 C CNN
@@
 L Device:R R6
 U 1 1 5C919740
-P 6650 1700
-F 0 "R6" H 6720 1746 50  0000 L CNN
-F 1 "R" H 6720 1655 50  0000 L CNN
-F 2 "Resistor_THT:R_Axial_DIN0207_L6.3mm_D2.5mm_P7.62mm_Horizontal" V 6580 1700 50  0001 C CNN
-F 3 "~" H 6650 1700 50  0001 C CNN
-	1    6650 1700
+P 6400 1700
+F 0 "R6" H 6470 1746 50  0000 L CNN
+F 1 "4.7K" H 6470 1655 50  0000 L CNN
+F 2 "Resistor_THT:R_Axial_DIN0207_L6.3mm_D2.5mm_P7.62mm_Horizontal" V 6330 1700 50  0001 C CNN
+F 3 "~" H 6400 1700 50  0001 C CNN
+	1    6400 1700
 	-1   0    0    1
 $EndComp
@@
 L Device:D D2
 U 1 1 5C91A5F5
-P 7050 2450
-F 0 "D2" H 7050 2666 50  0000 C CNN
-F 1 "D" H 7050 2575 50  0000 C CNN
-F 2 "Diode_THT:D_DO-35_SOD27_P7.62mm_Horizontal" H 7050 2450 50  0001 C CNN
-F 3 "~" H 7050 2450 50  0001 C CNN
-	1    7050 2450
-	-1   0    0    1
+P 7250 2400
+F 0 "D2" H 7250 2616 50  0000 C CNN
+F 1 "in916" H 7250 2525 50  0000 C CNN
+F 2 "Diode_THT:D_DO-35_SOD27_P7.62mm_Horizontal" H 7250 2400 50  0001 C CNN
+F 3 "~" H 7250 2400 50  0001 C CNN
+	1    7250 2400
+	0    1    1    0
 $EndComp
 $Comp
 L Device:D D1
 U 1 1 5C91BE51
-P 7050 2250
-F 0 "D1" H 7050 2466 50  0000 C CNN
-F 1 "D" H 7050 2375 50  0000 C CNN
-F 2 "Diode_THT:D_DO-35_SOD27_P7.62mm_Horizontal" H 7050 2250 50  0001 C CNN
-F 3 "~" H 7050 2250 50  0001 C CNN
-	1    7050 2250
-	1    0    0    -1
+P 7050 2400
+F 0 "D1" H 7050 2616 50  0000 C CNN
+F 1 "in916" H 7050 2525 50  0000 C CNN
+F 2 "Diode_THT:D_DO-35_SOD27_P7.62mm_Horizontal" H 7050 2400 50  0001 C CNN
+F 3 "~" H 7050 2400 50  0001 C CNN
+	1    7050 2400
+	0    -1   -1   0
 $EndComp
 $Comp
 L Device:R R2
 U 1 1 5C902560
-P 5750 2150
-F 0 "R2" V 5543 2150 50  0000 C CNN
-F 1 "R" V 5634 2150 50  0000 C CNN
-F 2 "Resistor_THT:R_Axial_DIN0207_L6.3mm_D2.5mm_P7.62mm_Horizontal" V 5680 2150 50  0001 C CNN
-F 3 "~" H 5750 2150 50  0001 C CNN
-	1    5750 2150
+P 5500 2150
+F 0 "R2" V 5293 2150 50  0000 C CNN
+F 1 "4.7K" V 5384 2150 50  0000 C CNN
+F 2 "Resistor_THT:R_Axial_DIN0207_L6.3mm_D2.5mm_P7.62mm_Horizontal" V 5430 2150 50  0001 C CNN
+F 3 "~" H 5500 2150 50  0001 C CNN
+	1    5500 2150
 	0    1    1    0
 $EndComp
@@
 	7350 3500 7700 3500
 $Comp
-L Transistor_FET:AO3401 Q3
+L Weather-rescue:AO3401-Transistor_FET Q3
 U 1 1 5C900ECB
 P 7250 4250
@@
 P 7050 4900
 F 0 "R8" H 7120 4946 50  0000 L CNN
-F 1 "R" H 7120 4855 50  0000 L CNN
+F 1 "20K" H 7120 4855 50  0000 L CNN
 F 2 "Resistor_THT:R_Axial_DIN0207_L6.3mm_D2.5mm_P7.62mm_Horizontal" V 6980 4900 50  0001 C CNN
 F 3 "~" H 7050 4900 50  0001 C CNN
@@
 Connection ~ 7700 3500
 Wire Wire Line
-	7700 3500 7950 3500
-Wire Wire Line
 	7700 3950 7950 3950
 Wire Wire Line
@@
 Connection ~ 7050 4250
 Wire Wire Line
-	6400 1350 6400 1850
+	6150 1350 6150 1850
 $Comp
 L Device:R R11
 U 1 1 5C914922
-P 7500 2350
-F 0 "R11" V 7293 2350 50  0000 C CNN
-F 1 "R" V 7384 2350 50  0000 C CNN
-F 2 "Resistor_THT:R_Axial_DIN0207_L6.3mm_D2.5mm_P7.62mm_Horizontal" V 7430 2350 50  0001 C CNN
-F 3 "~" H 7500 2350 50  0001 C CNN
-	1    7500 2350
+P 7600 2250
+F 0 "R11" V 7393 2250 50  0000 C CNN
+F 1 "3.3k" V 7484 2250 50  0000 C CNN
+F 2 "Resistor_THT:R_Axial_DIN0207_L6.3mm_D2.5mm_P7.62mm_Horizontal" V 7530 2250 50  0001 C CNN
+F 3 "~" H 7600 2250 50  0001 C CNN
+	1    7600 2250
 	0    1    1    0
 $EndComp
 Wire Wire Line
-	7650 2350 7950 2350
-Wire Wire Line
-	7950 2350 7950 3500
-Wire Wire Line
-	7200 2250 7200 2350
-Wire Wire Line
-	7350 2350 7200 2350
-Connection ~ 7200 2350
-Wire Wire Line
-	7200 2350 7200 2450
-Wire Wire Line
-	6900 2450 6900 2250
-Wire Wire Line
-	6900 2250 6600 2250
-Connection ~ 6900 2250
+	7250 2550 7150 2550
 $Comp
 L Device:R R9
 U 1 1 5C96EBEA
-P 6650 2650
-F 0 "R9" H 6720 2696 50  0000 L CNN
-F 1 "R" H 6720 2605 50  0000 L CNN
-F 2 "Resistor_THT:R_Axial_DIN0207_L6.3mm_D2.5mm_P7.62mm_Horizontal" V 6580 2650 50  0001 C CNN
-F 3 "~" H 6650 2650 50  0001 C CNN
-	1    6650 2650
-	1    0    0    -1
-$EndComp
-Wire Wire Line
-	5900 2150 6000 2150
-Wire Wire Line
-	6600 2050 6650 2050
-Wire Wire Line
-	7950 3500 8350 3500
-Connection ~ 7950 3500
+P 6400 2650
+F 0 "R9" H 6470 2696 50  0000 L CNN
+F 1 "4.7K" H 6470 2605 50  0000 L CNN
+F 2 "Resistor_THT:R_Axial_DIN0207_L6.3mm_D2.5mm_P7.62mm_Horizontal" V 6330 2650 50  0001 C CNN
+F 3 "~" H 6400 2650 50  0001 C CNN
+	1    6400 2650
+	1    0    0    -1
+$EndComp
+Wire Wire Line
+	5650 2150 5750 2150
+Wire Wire Line
+	6350 2050 6400 2050
 Wire Wire Line
 	7950 3950 8350 3950
@@
 Connection ~ 4600 3650
 Wire Wire Line
-	3850 2850 4600 2850
-Wire Wire Line
 	4600 2850 4600 3250
 Connection ~ 4600 3250
@@
 	4900 4250 4900 2150
 Wire Wire Line
-	4900 2150 5600 2150
-Wire Wire Line
-	6400 2450 6400 2850
-Wire Wire Line
-	6400 2850 4600 2850
+	6150 2450 6150 2850
+Wire Wire Line
+	6150 2850 4600 2850
+Wire Wire Line
+	3850 3050 5300 3050
+Wire Wire Line
+	5300 3050 5300 1350
+Wire Wire Line
+	6150 2850 6400 2850
+Wire Wire Line
+	6400 2850 6400 2800
+Connection ~ 6150 2850
+Wire Wire Line
+	6400 2500 6400 2050
+Wire Wire Line
+	6150 1350 6400 1350
+Wire Wire Line
+	6400 1350 6400 1550
+Connection ~ 6150 1350
+Wire Wire Line
+	6400 1850 6400 2050
+Connection ~ 6400 2050
+Wire Wire Line
+	7050 2250 7250 2250
+Wire Wire Line
+	7700 3500 7950 3500
+Wire Wire Line
+	7150 2550 7150 2850
+Connection ~ 7150 2550
+Wire Wire Line
+	7150 2550 7050 2550
+Wire Wire Line
+	7750 2250 7950 2250
+Wire Wire Line
+	7950 2250 7950 3500
+Connection ~ 7950 3500
+Wire Wire Line
+	7950 3500 8350 3500
+Wire Wire Line
+	7250 2250 7450 2250
+Connection ~ 7250 2250
+$Comp
+L Device:C C?
+U 1 1 5C96A149
+P 6650 2250
+F 0 "C?" V 6398 2250 50  0000 C CNN
+F 1 "C" V 6489 2250 50  0000 C CNN
+F 2 "" H 6688 2100 50  0001 C CNN
+F 3 "~" H 6650 2250 50  0001 C CNN
+	1    6650 2250
+	0    1    1    0
+$EndComp
+Text Label 7150 2850 0    50   ~ 0
+0v
+Text Label 6150 1300 0    50   ~ 0
+5v
+Wire Wire Line
+	4900 2150 5350 2150
+Wire Wire Line
+	5300 1350 6150 1350
+Wire Wire Line
+	3850 2850 4600 2850
 Connection ~ 4600 2850
 Wire Wire Line
-	3850 3050 5300 3050
-Wire Wire Line
-	5300 3050 5300 1350
-Wire Wire Line
-	5300 1350 6400 1350
-Wire Wire Line
-	6400 2850 6650 2850
-Wire Wire Line
-	6650 2850 6650 2800
+	6350 2250 6500 2250
+Wire Wire Line
+	6800 2250 7050 2250
+Connection ~ 7050 2250
+Wire Wire Line
+	6400 2850 7150 2850
 Connection ~ 6400 2850
-Wire Wire Line
-	6650 2500 6650 2050
-Wire Wire Line
-	6400 1350 6650 1350
-Wire Wire Line
-	6650 1350 6650 1550
-Connection ~ 6400 1350
-Wire Wire Line
-	6650 1850 6650 2050
-Connection ~ 6650 2050
+Text Label 5750 3400 0    50   ~ 0
+24v
 $EndSCHEMATC

Commit message: schematic changes
Parts:
- added R11, R7: 4.7K, symbol Device:R
- C4: renamed from C?; value C -> 0.1uF
- gave numbers to parts that had none: 2
- renumbered R9 to R10, R7 to R12, R8 to R13, R10 to R14, R12 to R15, R11 to R16, R1 to R3, R2 to R4, R3 to R5, R4 to R6, R5 to R8, R6 to R9, U1 to U5
Connections:
- net labels added: Vdrive
- wire segments 73 -> 86
Other:
- moved on the sheet: C4, D1, D2, R16

Commit message: Start PCB
Parts:
- C4: footprint (none) -> Capacitor_THT:C_Disc_D3.8mm_W2.6mm_P2.50mm
- J2, J3: footprint (none) -> Connector_PinHeader_2.54mm:PinHeader_1x04_P2.54mm_Vertical
- R11, R7: footprint (none) -> Resistor_THT:R_Axial_DIN0207_L6.3mm_D2.5mm_P7.62mm_Horizontal
Connections:
- net labels added: GNDS
Other:
- moved on the sheet: Q2, R5
Changed lines of the file:
@@
 L Weather-rescue:AO3401-Transistor_FET Q2
 U 1 1 5C8F913C
-P 6300 3600
-F 0 "Q2" V 6643 3600 50  0000 C CNN
-F 1 "AO3401" V 6552 3600 50  0000 C CNN
-F 2 "Package_TO_SOT_SMD:SOT-23" H 6500 3525 50  0001 L CIN
-F 3 "" H 6300 3600 50  0001 L CNN
-	1    6300 3600
+P 6300 3550
+F 0 "Q2" V 6643 3550 50  0000 C CNN
+F 1 "AO3401" V 6552 3550 50  0000 C CNN
+F 2 "Package_TO_SOT_SMD:SOT-23" H 6500 3475 50  0001 L CIN
+F 3 "" H 6300 3550 50  0001 L CNN
+	1    6300 3550
 	0    1    -1   0
 $EndComp
@@
 L Device:R R5
 U 1 1 5C91429E
-P 5750 3750
-F 0 "R5" H 5820 3796 50  0000 L CNN
-F 1 "2.2k" H 5820 3705 50  0000 L CNN
-F 2 "Resistor_THT:R_Axial_DIN0207_L6.3mm_D2.5mm_P7.62mm_Horizontal" V 5680 3750 50  0001 C CNN
-F 3 "~" H 5750 3750 50  0001 C CNN
-	1    5750 3750
+P 5750 3700
+F 0 "R5" H 5820 3746 50  0000 L CNN
+F 1 "2.2k" H 5820 3655 50  0000 L CNN
+F 2 "Resistor_THT:R_Axial_DIN0207_L6.3mm_D2.5mm_P7.62mm_Horizontal" V 5680 3700 50  0001 C CNN
+F 3 "~" H 5750 3700 50  0001 C CNN
+	1    5750 3700
 	1    0    0    -1
 $EndComp
@@
 	6300 4300 6300 4600
 Wire Wire Line
-	6300 3800 6300 3950
-Wire Wire Line
-	5750 3500 6100 3500
-Wire Wire Line
-	5750 3600 5750 3500
-Wire Wire Line
-	5750 3900 5750 3950
+	5750 3450 6100 3450
+Wire Wire Line
+	5750 3550 5750 3450
 Wire Wire Line
 	5750 3950 6300 3950
@@
 Connection ~ 7350 5650
 Wire Wire Line
-	6500 3500 7050 3500
-Wire Wire Line
-	7350 4050 7350 3500
-Connection ~ 7350 3500
-Wire Wire Line
-	7350 3500 7700 3500
+	6500 3450 7050 3450
+Wire Wire Line
+	7350 4000 7350 3450
+Connection ~ 7350 3450
+Wire Wire Line
+	7350 3450 7700 3450
 $Comp
 L Weather-rescue:AO3401-Transistor_FET Q3
@@
 Wire Wire Line
 	7050 5650 7350 5650
-Wire Wire Line
-	7700 3650 7700 3500
-Connection ~ 7700 3500
+Connection ~ 7700 3450
 Wire Wire Line
 	7700 3950 7950 3950
@@
 	7950 3950 7950 5650
 Wire Wire Line
-	7050 3750 7050 3500
-Connection ~ 7050 3500
-Wire Wire Line
-	7050 3500 7350 3500
+	7050 3700 7050 3450
+Connection ~ 7050 3450
+Wire Wire Line
+	7050 3450 7350 3450
 Wire Wire Line
 	7050 4050 7050 4250
@@
 Connection ~ 7950 3950
 Wire Wire Line
-	3850 3450 5750 3450
-Wire Wire Line
-	5750 3450 5750 3500
-Connection ~ 5750 3500
-Wire Wire Line
 	3850 4050 4600 4050
 Wire Wire Line
@@
 	7200 2250 7400 2250
 Wire Wire Line
-	7700 3500 7950 3500
+	7700 3450 7950 3450
 Wire Wire Line
 	7300 2550 7300 2850
@@
 	7900 2250 7950 2250
 Wire Wire Line
-	7950 2250 7950 3500
-Connection ~ 7950 3500
-Wire Wire Line
-	7950 3500 8350 3500
+	7950 2200 7950 2250
+Connection ~ 7950 3450
 Wire Wire Line
 	7400 2250 7600 2250
@@
 F 0 "C4" V 6648 2250 50  0000 C CNN
 F 1 "0.1uF" V 6739 2250 50  0000 C CNN
-F 2 "" H 6938 2100 50  0001 C CNN
+F 2 "Capacitor_THT:C_Disc_D3.8mm_W2.6mm_P2.50mm" H 6938 2100 50  0001 C CNN
 F 3 "~" H 6900 2250 50  0001 C CNN
 	1    6900 2250
@@
 	3850 2850 4600 2850
 Connection ~ 4600 2850
-Text Label 5750 3400 0    50   ~ 0
+Text Label 5800 3450 0    50   ~ 0
 24v
 $Comp
@@
 F 0 "R11" V 6393 2250 50  0000 C CNN
 F 1 "4.7K" V 6484 2250 50  0000 C CNN
-F 2 "" V 6530 2250 50  0001 C CNN
+F 2 "Resistor_THT:R_Axial_DIN0207_L6.3mm_D2.5mm_P7.62mm_Horizontal" V 6530 2250 50  0001 C CNN
 F 3 "~" H 6600 2250 50  0001 C CNN
 	1    6600 2250
@@
 F 0 "R7" V 5693 2500 50  0000 C CNN
 F 1 "4.7K" V 5784 2500 50  0000 C CNN
-F 2 "" V 5830 2500 50  0001 C CNN
+F 2 "Resistor_THT:R_Axial_DIN0207_L6.3mm_D2.5mm_P7.62mm_Horizontal" V 5830 2500 50  0001 C CNN
 F 3 "~" H 5900 2500 50  0001 C CNN
 	1    5900 2500
@@
 	3850 3250 3700 3250
 Connection ~ 3850 3250
-Wire Wire Line
-	3850 3450 3700 3450
-Connection ~ 3850 3450
 Wire Wire Line
 	3850 3650 3700 3650
@@
 F 0 "J3" H 3900 2950 50  0000 L CNN
 F 1 "4_Way_Wire" H 3750 2800 50  0000 L CNN
-F 2 "" H 3850 3700 50  0001 C CNN
+F 2 "Connector_PinHeader_2.54mm:PinHeader_1x04_P2.54mm_Vertical" H 3850 3700 50  0001 C CNN
 F 3 "" H 3850 3700 50  0001 C CNN
 	1    3950 3650
@@
 F 0 "J2" H 3900 3000 50  0000 L CNN
 F 1 "4_Way_Wire" H 3800 3100 50  0000 L CNN
-F 2 "" H 3850 2900 50  0001 C CNN
+F 2 "Connector_PinHeader_2.54mm:PinHeader_1x04_P2.54mm_Vertical" H 3850 2900 50  0001 C CNN
 F 3 "" H 3850 2900 50  0001 C CNN
 	1    3950 2850
@@
 L power:Vdrive #PWR02
 U 1 1 5C99BC4B
-P 8350 3500
-F 0 "#PWR02" H 8150 3350 50  0001 C CNN
-F 1 "Vdrive" H 8367 3673 50  0000 C CNN
-F 2 "" H 8350 3500 50  0001 C CNN
-F 3 "" H 8350 3500 50  0001 C CNN
-	1    8350 3500
-	1    0    0    -1
-$EndComp
+P 8350 3450
+F 0 "#PWR02" H 8150 3300 50  0001 C CNN
+F 1 "Vdrive" H 8367 3623 50  0000 C CNN
+F 2 "" H 8350 3450 50  0001 C CNN
+F 3 "" H 8350 3450 50  0001 C CNN
+	1    8350 3450
+	1    0    0    -1
+$EndComp
+Connection ~ 7950 2250
+Wire Wire Line
+	7950 2250 7950 3450
+Wire Wire Line
+	7700 3450 7700 3650
+Wire Wire Line
+	5750 3850 5750 3950
+Wire Wire Line
+	6300 3750 6300 3950
+Wire Wire Line
+	3700 3450 3850 3450
+Connection ~ 5750 3450
+Connection ~ 3850 3450
+Wire Wire Line
+	3850 3450 5750 3450
+Wire Wire Line
+	7950 3450 8350 3450
+$Comp
+L power:GNDS #PWR0101
+U 1 1 5CFCB28B
+P 8350 3950
+F 0 "#PWR0101" H 8350 3700 50  0001 C CNN
+F 1 "GNDS" H 8355 3777 50  0000 C CNN
+F 2 "" H 8350 3950 50  0001 C CNN
+F 3 "" H 8350 3950 50  0001 C CNN
+	1    8350 3950
+	1    0    0    -1
+$EndComp

Commit message: small compnent changes
Connections:
- wire segments 86 -> 85
